File: quicklogic-quick-feather-board.sch (KiCad schematic (older format))
At the start: 89 parts, among them IC1 EOS-S3, J1 825437-4, J2 1x12_pinhead, J3 1x16_pinhead, J4 S2B-PH-SM4-TB_LF__SN_, J5 0473460001, J6 FTSH-105-01-L-DV-K, Q1 RV1C002UN, Q2 RV1C001ZP, Q3 RV1C002UN, Q4 RV1C002UN, Q5 RV1C002UN, U1 TPS62821DLCR, U2 MCP73831T-2ACI_OT, U3 GD25Q16CWIGR, U4 DPS310, U5 MC3635, X1 ECS-_327-12_5-34B-TR

Commit message: R22 marked as DNP
Parts:
- R22: Populate (none) -> DNP
Other:
- note added: "DNP"
Changed lines of the file:
@@
 F 5 "CRCW040210K0FKEDHP" H 7650 3300 60  0001 L CNN "MPN"
 F 6 "10k" H 7350 2800 50  0000 L CNN "Val"
+F 7 "DNP" H 7450 3000 50  0001 C CNN "Populate"
 	1    7450 3000
 	0    -1   -1   0
@@
 Text Label 5500 2150 0    50   ~ 0
 IMU_INT
+Text Notes 7500 3100 1    51   ~ 10
+DNP
 $EndSCHEMATC

Commit message: Added a 2-pin header to configure bootstrap pins for EOS IC
Parts:
- added J7: S2B-PH-SM4-TB_LF__SN_, quicklogic-quick-feather-board-footprints:PinHeader_2x1mm_P2mm_SMD_RA, symbol quicklogic-quick-feather-board:S2B-PH-SM4-TB_LF__SN_
- R22: DNP (none) -> 1; Populate DNP -> (none)
Connections:
- wire segments 304 -> 307
Changed lines of the file:
@@
 F 5 "CRCW040210K0FKEDHP" H 7650 3300 60  0001 L CNN "MPN"
 F 6 "10k" H 7350 2800 50  0000 L CNN "Val"
-F 7 "DNP" H 7450 3000 50  0001 C CNN "Populate"
+F 7 "1" H 7450 3000 50  0001 C CNN "DNP"
 	1    7450 3000
 	0    -1   -1   0
@@
 L quicklogic-quick-feather-board:+3V3 #PWR016
 U 1 1 5DEB4A46
-P 7450 2350
-F 0 "#PWR016" H 7450 2350 50  0001 C CNN
-F 1 "+3V3" H 7435 2473 50  0000 C CNN
-F 2 "" H 7450 2350 50  0001 C CNN
-F 3 "" H 7450 2350 50  0001 C CNN
-	1    7450 2350
-	1    0    0    -1
-$EndComp
-Text Notes 7100 2100 0    50   ~ 0
+P 7800 2200
+F 0 "#PWR016" H 7800 2200 50  0001 C CNN
+F 1 "+3V3" H 7785 2323 50  0000 C CNN
+F 2 "" H 7800 2200 50  0001 C CNN
+F 3 "" H 7800 2200 50  0001 C CNN
+	1    7800 2200
+	1    0    0    -1
+$EndComp
+Text Notes 7150 3650 0    50   ~ 0
 Mount R23 for debug mode, \notherwise R22
 Wire Wire Line
@@
 Text Notes 7500 3100 1    51   ~ 10
 DNP
+$Comp
+L quicklogic-quick-feather-board:S2B-PH-SM4-TB_LF__SN_ J7
+U 1 1 5DFAC16F
+P 7450 2050
+F 0 "J7" V 7225 2058 50  0000 C CNN
+F 1 "S2B-PH-SM4-TB_LF__SN_" V 7316 2058 50  0000 C CNN
+F 2 "quicklogic-quick-feather-board-footprints:PinHeader_2x1mm_P2mm_SMD_RA" H 7650 2250 60  0001 L CNN
+F 3 "http://www.jst-mfg.com/product/pdf/eng/ePH.pdf" H 7650 2350 60  0001 L CNN
+F 4 "S2B-PH-SM4-TB(LF)(SN)" H 7650 2550 60  0001 L CNN "MPN"
+F 5 "JST Sales America Inc." H 7650 3150 60  0001 L CNN "Manufacturer"
+	1    7450 2050
+	1    0    0    1
+$EndComp
+Wire Wire Line
+	7450 2400 7450 2150
+Wire Wire Line
+	7550 2150 7550 2250
+Wire Wire Line
+	7550 2250 7800 2250
 $EndSCHEMATC

Commit message: Updated component definitions on PCB
Parts:
- removed J7: S2B-PH-SM4-TB_LF__SN_, quicklogic-quick-feather-board-footprints:PinHeader_2x1mm_P2mm_SMD_RA, symbol quicklogic-quick-feather-board:S2B-PH-SM4-TB_LF__SN_
- added J7: 22-23-2021, antmicro-footprints:PinHeader_1x2_P2.54mm_Drill1.02mm, symbol quicklogic-quick-feather-board:22-23-2021
Changed lines of the file:
@@
 Text Notes 7500 3100 1    51   ~ 10
 DNP
-$Comp
-L quicklogic-quick-feather-board:S2B-PH-SM4-TB_LF__SN_ J7
-U 1 1 5DFAC16F
-P 7450 2050
-F 0 "J7" V 7225 2058 50  0000 C CNN
-F 1 "S2B-PH-SM4-TB_LF__SN_" V 7316 2058 50  0000 C CNN
-F 2 "quicklogic-quick-feather-board-footprints:PinHeader_2x1mm_P2mm_SMD_RA" H 7650 2250 60  0001 L CNN
-F 3 "http://www.jst-mfg.com/product/pdf/eng/ePH.pdf" H 7650 2350 60  0001 L CNN
-F 4 "S2B-PH-SM4-TB(LF)(SN)" H 7650 2550 60  0001 L CNN "MPN"
-F 5 "JST Sales America Inc." H 7650 3150 60  0001 L CNN "Manufacturer"
-	1    7450 2050
-	1    0    0    1
-$EndComp
 Wire Wire Line
 	7450 2400 7450 2150
@@
 Wire Wire Line
 	7550 2250 7800 2250
+$Comp
+L quicklogic-quick-feather-board:22-23-2021 J7
+U 1 1 5E0462F0
+P 7550 2050
+F 0 "J7" H 7700 1800 50  0000 R CNN
+F 1 "22-23-2021" H 7700 1900 50  0000 R CNN
+F 2 "antmicro-footprints:PinHeader_1x2_P2.54mm_Drill1.02mm" H 7750 2250 60  0001 L CNN
+F 3 "https://media.digikey.com/pdf/Data%20Sheets/Molex%20PDFs/A-6373-N_Series_Dwg_2010-12-03.pdf" H 7750 2350 60  0001 L CNN
+F 4 "22-23-2021" H 7750 2550 60  0001 L CNN "MPN"
+F 5 "Molex" H 7750 3150 60  0001 L CNN "Manufacturer"
+	1    7550 2050
+	-1   0    0    1
+$EndComp
 $EndSCHEMATC

Commit message: EOS-S3 changed to QFN version
Parts:
- removed IC1: EOS-S3, quicklogic-quick-feather-board-footprints:42-WLCSP, symbol quicklogic-quick-feather-board:EOS-S3
- added IC1: EOS-S3-QFN, quicklogic-quick-feather-board-footprints:QFN-64_EP_8.5x8.5_EOS, symbol quicklogic-quick-feather-board:EOS-S3-QFN
- R12, R17: footprint quicklogic-quick-feather-board-footprints:0402 -> quicklogic-quick-feather-board-footprints:0402-res
Connections:
- wire segments 307 -> 312
Changed lines of the file:
@@
 EESchema Schematic File Version 4
+LIBS:quicklogic-quick-feather-board-cache
 EELAYER 30 0
 EELAYER END
@@
 $EndComp
 $Comp
-L quicklogic-quick-feather-board:EOS-S3 IC1
-U 1 1 5DCF18DD
-P 3300 1400
-F 0 "IC1" H 4225 1565 50  0000 C CNN
-F 1 "EOS-S3" H 4225 1474 50  0000 C CNN
-F 2 "quicklogic-quick-feather-board-footprints:42-WLCSP" H 4950 -1700 50  0001 C CNN
-F 3 "" H 5050 -1600 50  0001 C CNN
-	1    3300 1400
-	1    0    0    -1
-$EndComp
-$Comp
 L quicklogic-quick-feather-board:DFE201610E-R47M=P2 L1
 U 1 1 5DC19811
@@
 L quicklogic-quick-feather-board:GND #PWR03
 U 1 1 5DC5B39C
-P 2800 4300
-F 0 "#PWR03" H 2800 4050 50  0001 C CNN
-F 1 "GND" H 2805 4127 50  0000 C CNN
-F 2 "" H 2800 4300 50  0001 C CNN
-F 3 "" H 2800 4300 50  0001 C CNN
-	1    2800 4300
+P 2800 3400
+F 0 "#PWR03" H 2800 3150 50  0001 C CNN
+F 1 "GND" H 2805 3227 50  0000 C CNN
+F 2 "" H 2800 3400 50  0001 C CNN
+F 3 "" H 2800 3400 50  0001 C CNN
+	1    2800 3400
 	1    0    0    -1
 $EndComp
@@
 Connection ~ 2800 3100
 Wire Wire Line
-	2800 3100 2800 3200
-Wire Wire Line
-	3200 3200 2800 3200
-Connection ~ 2800 3200
-Wire Wire Line
-	2800 3200 2800 3300
-Wire Wire Line
 	3200 3300 2800 3300
 Connection ~ 2800 3300
@@
 Connection ~ 2800 3400
 Wire Wire Line
-	2800 3400 2800 4300
-Wire Wire Line
 	3200 1550 2900 1550
 Wire Wire Line
@@
 Connection ~ 2900 1550
 Wire Wire Line
-	3200 1850 2900 1850
-Wire Wire Line
-	2900 1850 2900 1700
-Connection ~ 2900 1700
-Wire Wire Line
-	3200 1950 2900 1950
-Wire Wire Line
-	2900 1950 2900 1850
-Connection ~ 2900 1850
-Wire Wire Line
 	3200 2400 2550 2400
 $Comp
@@
 $EndComp
 $Comp
-L quicklogic-quick-feather-board:TP_SMD1MM TP1
-U 1 1 5DC6A7F5
-P 2750 2150
-F 0 "TP1" V 2750 2050 50  0000 C CNN
-F 1 "TP_SMD1MM" H 2750 2050 50  0001 C CNN
-F 2 "quicklogic-quick-feather-board-footprints:Testpoint_smd_1mm" H 2950 2350 60  0001 L CNN
-F 3 "" H 2950 2450 60  0001 L CNN
-F 4 "N/A" H 0   0   50  0001 C CNN "MPN"
-F 5 "N/A" H 0   0   50  0001 C CNN "Manufacturer"
-	1    2750 2150
-	0    1    1    0
-$EndComp
-$Comp
-L quicklogic-quick-feather-board:TP_SMD1MM TP2
-U 1 1 5DC6A90F
-P 2750 2250
-F 0 "TP2" V 2750 2150 50  0000 C CNN
-F 1 "TP_SMD1MM" H 2750 2150 50  0001 C CNN
-F 2 "quicklogic-quick-feather-board-footprints:Testpoint_smd_1mm" H 2950 2450 60  0001 L CNN
-F 3 "" H 2950 2550 60  0001 L CNN
-F 4 "N/A" H 0   0   50  0001 C CNN "MPN"
-F 5 "N/A" H 0   0   50  0001 C CNN "Manufacturer"
-	1    2750 2250
-	0    1    1    0
-$EndComp
-Wire Wire Line
-	3200 2150 2850 2150
-Wire Wire Line
-	2850 2250 3200 2250
-$Comp
 L quicklogic-quick-feather-board:ECS-_327-12_5-34B-TR X1
 U 1 1 5DC7219A
@@
 F 0 "R17" V 6755 7170 60  0000 L CNN
 F 1 "R_100k_1%_0402" H 6800 6950 60  0001 C CNN
-F 2 "quicklogic-quick-feather-board-footprints:0402" H 7000 7300 60  0001 L CNN
+F 2 "quicklogic-quick-feather-board-footprints:0402-res" H 7000 7300 60  0001 L CNN
 F 3 "" H 6800 7100 50  0001 C CNN
 F 4 "PANASONIC" H 7000 7500 60  0001 L CNN "Manufacturer"
@@
 F 0 "R12" V 5805 6120 60  0000 L CNN
 F 1 "R_100k_1%_0402" H 5850 5900 60  0001 C CNN
-F 2 "quicklogic-quick-feather-board-footprints:0402" H 6050 6250 60  0001 L CNN
+F 2 "quicklogic-quick-feather-board-footprints:0402-res" H 6050 6250 60  0001 L CNN
 F 3 "" H 5850 6050 50  0001 C CNN
 F 4 "PANASONIC" H 6050 6450 60  0001 L CNN "Manufacturer"
@@
 $EndComp
 Connection ~ 4400 6450
-Text Notes 3300 4650 0    50   ~ 0
+Text Notes 5950 4750 0    50   ~ 0
 Maximum power consumption for A and B rails:\nLDO mode: 65mA (VCCIOA) 114mA (VCCIOB)\nLDO bypass mode: 77mA (VCCIOA) 269mA (VCCIOB)
 $Comp
@@
 Wire Wire Line
 	1600 4500 1850 4500
-Text Notes 3300 5000 0    50   ~ 0
+Text Notes 5950 5100 0    50   ~ 0
 The multi-functional IOs have four programmable drive \nstrength states: 2 mA, 4 mA, 8 mA, 12 mA \n(refer to datasheet page 92)
 Text Notes 10150 2400 0    50   ~ 0
@@
 	1    0    0    -1
 $EndComp
-Text Label 2850 2150 0    50   ~ 0
-VDD1
 Text Label 1650 1400 1    50   ~ 0
 VDD2
-Text Label 2850 2250 0    50   ~ 0
-VDD2
 Text Label 1950 1400 1    50   ~ 0
 VDD1
@@
 	-1   0    0    1
 $EndComp
+Wire Wire Line
+	2850 2250 3200 2250
+$Comp
+L quicklogic-quick-feather-board:TP_SMD1MM TP2
+U 1 1 5DC6A90F
+P 2750 2250
+F 0 "TP2" V 2750 2150 50  0000 C CNN
+F 1 "TP_SMD1MM" H 2750 2150 50  0001 C CNN
+F 2 "quicklogic-quick-feather-board-footprints:Testpoint_smd_1mm" H 2950 2450 60  0001 L CNN
+F 3 "" H 2950 2550 60  0001 L CNN
+F 4 "N/A" H 0   0   50  0001 C CNN "MPN"
+F 5 "N/A" H 0   0   50  0001 C CNN "Manufacturer"
+	1    2750 2250
+	0    1    1    0
+$EndComp
+Text Label 2850 2250 0    50   ~ 0
+VDD2
+Text Label 2850 2150 0    50   ~ 0
+VDD1
+Wire Wire Line
+	3200 2150 2850 2150
+$Comp
+L quicklogic-quick-feather-board:TP_SMD1MM TP1
+U 1 1 5DC6A7F5
+P 2750 2150
+F 0 "TP1" V 2750 2050 50  0000 C CNN
+F 1 "TP_SMD1MM" H 2750 2050 50  0001 C CNN
+F 2 "quicklogic-quick-feather-board-footprints:Testpoint_smd_1mm" H 2950 2350 60  0001 L CNN
+F 3 "" H 2950 2450 60  0001 L CNN
+F 4 "N/A" H 0   0   50  0001 C CNN "MPN"
+F 5 "N/A" H 0   0   50  0001 C CNN "Manufacturer"
+	1    2750 2150
+	0    1    1    0
+$EndComp
+$Comp
+L quicklogic-quick-feather-board:EOS-S3-QFN IC1
+U 1 1 5E0610BF
+P 3300 1400
+F 0 "IC1" H 4225 2265 50  0000 C CNN
+F 1 "EOS-S3-QFN" H 4225 2174 50  0000 C CNN
+F 2 "quicklogic-quick-feather-board-footprints:QFN-64_EP_8.5x8.5_EOS" H 4250 -1900 50  0001 C CNN
+F 3 "" H 5050 -1600 50  0001 C CNN
+	1    3300 1400
+	1    0    0    -1
+$EndComp
+Wire Wire Line
+	3200 1800 2900 1800
+Wire Wire Line
+	2900 1800 2900 1700
+Connection ~ 2900 1700
+Wire Wire Line
+	2900 850  3200 850
+Wire Wire Line
+	2900 950  3200 950
+Connection ~ 2900 950
+Wire Wire Line
+	2900 950  2900 850
+Wire Wire Line
+	3200 1150 2900 1150
+Connection ~ 2900 1150
+Wire Wire Line
+	2900 1150 2900 950
+Wire Wire Line
+	3200 1250 2900 1250
+Connection ~ 2900 1250
+Wire Wire Line
+	2900 1250 2900 1150
+Wire Wire Line
+	3200 1350 2900 1350
+Wire Wire Line
+	2900 1250 2900 1350
+Connection ~ 2900 1350
+Wire Wire Line
+	2900 1350 2900 1550
+Wire Wire Line
+	2800 3100 2800 3300
 $EndSCHEMATC

Commit message: Changed jumper to mini jumper + slide switch. Footprint update
Parts:
- removed J7: 22-23-2021, antmicro-footprints:PinHeader_1x2_P2.54mm_Drill1.02mm, symbol quicklogic-quick-feather-board:22-23-2021
- added J7: MC-HVT1-S02-G, quicklogic-quick-feather-board-footprints:PinHeader_1x2_P1.27mm_Drill.7mm_with_622002115121_plug, symbol quicklogic-quick-feather-board:MC-HVT1-S02-G
- added S3: MSS3-V-T_R, quicklogic-quick-feather-board-footprints:Switch_Slide_MSS3, symbol quicklogic-quick-feather-board:MSS3-V-T_R
Connections:
- wire segments 312 -> 316
Changed lines of the file:
@@
 DNP
 Wire Wire Line
-	7450 2400 7450 2150
+	7450 2400 7450 2250
 Wire Wire Line
 	7550 2150 7550 2250
 Wire Wire Line
 	7550 2250 7800 2250
-$Comp
-L quicklogic-quick-feather-board:22-23-2021 J7
-U 1 1 5E0462F0
-P 7550 2050
-F 0 "J7" H 7700 1800 50  0000 R CNN
-F 1 "22-23-2021" H 7700 1900 50  0000 R CNN
-F 2 "antmicro-footprints:PinHeader_1x2_P2.54mm_Drill1.02mm" H 7750 2250 60  0001 L CNN
-F 3 "https://media.digikey.com/pdf/Data%20Sheets/Molex%20PDFs/A-6373-N_Series_Dwg_2010-12-03.pdf" H 7750 2350 60  0001 L CNN
-F 4 "22-23-2021" H 7750 2550 60  0001 L CNN "MPN"
-F 5 "Molex" H 7750 3150 60  0001 L CNN "Manufacturer"
-	1    7550 2050
-	-1   0    0    1
-$EndComp
 Wire Wire Line
 	2850 2250 3200 2250
@@
 Wire Wire Line
 	2800 3100 2800 3300
+$Comp
+L quicklogic-quick-feather-board:MC-HVT1-S02-G J7
+U 1 1 5E00A4C3
+P 7550 2000
+F 0 "J7" H 7450 1900 50  0000 R CNN
+F 1 "MC-HVT1-S02-G" H 7450 2000 50  0000 R CNN
+F 2 "quicklogic-quick-feather-board-footprints:PinHeader_1x2_P1.27mm_Drill.7mm_with_622002115121_plug" H 7750 2300 60  0001 L CNN
+F 3 "http://www.farnell.com/datasheets/2605295.pdf" H 7750 2400 60  0001 L CNN
+F 4 "MC-HVT1-S02-G" H 7750 2500 60  0001 L CNN "MPN"
+F 5 "Multicomp" H 7750 2600 60  0001 L CNN "Manufacturer"
+	1    7550 2000
+	-1   0    0    1
+$EndComp
+$Comp
+L quicklogic-quick-feather-board:MSS3-V-T_R S3
+U 1 1 5E00B30F
+P 7600 1600
+F 0 "S3" H 7600 1881 50  0000 C CNN
+F 1 "MSS3-V-T_R" H 7600 1790 50  0000 C CNN
+F 2 "quicklogic-quick-feather-board-footprints:Switch_Slide_MSS3" H 7800 1800 50  0001 L CNN
+F 3 "https://pl.mouser.com/datasheet/2/910/605_MSS34-1571494.pdf" H 7800 1900 60  0001 L CNN
+F 4 "MSS3-V-T/R" H 7800 2100 60  0001 L CNN "MPN"
+F 5 "Diptronics" H 7800 2220 60  0001 L CNN "Manufacturer"
+	1    7600 1600
+	1    0    0    -1
+$EndComp
+$Comp
+L quicklogic-quick-feather-board:+3V3 #PWR0136
+U 1 1 5E01BEDD
+P 7850 1500
+F 0 "#PWR0136" H 7850 1500 50  0001 C CNN
+F 1 "+3V3" H 7835 1623 50  0000 C CNN
+F 2 "" H 7850 1500 50  0001 C CNN
+F 3 "" H 7850 1500 50  0001 C CNN
+	1    7850 1500
+	0    1    1    0
+$EndComp
+Wire Wire Line
+	7450 2250 7250 2250
+Wire Wire Line
+	7250 2250 7250 1600
+Wire Wire Line
+	7250 1600 7400 1600
+Connection ~ 7450 2250
+Wire Wire Line
+	7450 2250 7450 2150
 $EndSCHEMATC

Commit message: Placement proposal
Parts:
- removed D4: UHD1110-FKA, quicklogic-quick-feather-board-footprints:LED-RGB-5DS-UHD1110-FKA, symbol quicklogic-quick-feather-board:UHD1110-FKA
- removed J7: MC-HVT1-S02-G, quicklogic-quick-feather-board-footprints:PinHeader_1x2_P1.27mm_Drill.7mm_with_622002115121_plug, symbol quicklogic-quick-feather-board:MC-HVT1-S02-G
- removed Q1, Q3, Q4, Q5: RV1C002UN, quicklogic-quick-feather-board-footprints:VML0806, symbol quicklogic-quick-feather-board:RV1C002UN
- removed Q2: RV1C001ZP, quicklogic-quick-feather-board-footprints:VML0806, symbol quicklogic-quick-feather-board:RV1C001ZP
- removed S3: MSS3-V-T_R, quicklogic-quick-feather-board-footprints:Switch_Slide_MSS3, symbol quicklogic-quick-feather-board:MSS3-V-T_R
- added D4: ASMB-MTB1-0A3A2, quicklogic-quick-feather-board-footprints:LED-PLCC4_3.2x2.8mm, symbol quicklogic-quick-feather-board:ASMB-MTB1-0A3A2
- added J7: 22-23-2021, quicklogic-quick-feather-board-footprints:PinHeader_1x2_P2.54_Drill0.9mm, symbol quicklogic-quick-feather-board:22-23-2021
- added Q1: NX3008CBKV, quicklogic-quick-feather-board-footprints:SOT-563, symbol quicklogic-quick-feather-board:NX3008CBKV
- added Q2, Q3: 2N7002PV, quicklogic-quick-feather-board-footprints:SOT-563, symbol quicklogic-quick-feather-board:2N7002PV
Connections:
- net labels removed: SDW_IO
- wire segments 316 -> 317
Other:
- moved on the sheet: R16, R24, R26

Commit message: Added J8 connector, extended board outline
Parts:
- removed J1: 825437-4, quicklogic-quick-feather-board-footprints:TE_825437-4, symbol quicklogic-quick-feather-board:825437-4
- added J1: 22-23-2021, quicklogic-quick-feather-board-footprints:PinHeader_1x2_P2.54_Drill0.9mm, symbol quicklogic-quick-feather-board:22-23-2021
- added J8: 2x8_pinhead, quicklogic-quick-feather-board-footprints:2x8_pinhead, symbol quicklogic-quick-feather-board:2x8_pinhead
- added M1, M2, M3, M4: mounting_pad, quicklogic-quick-feather-board-footprints:MPAD, symbol quicklogic-quick-feather-board:mounting_pad
- added R31: R_10k_0402, quicklogic-quick-feather-board-footprints:0402-res, symbol quicklogic-quick-feather-board:R_10k_0402
- added R33, R41, R42: EXB2HV220JV, quicklogic-quick-feather-board-footprints:R_Array_Convex_8x0602, symbol quicklogic-quick-feather-board:EXB2HV220JV
- added R38, R39, R40: R_22R_0402, quicklogic-quick-feather-board-footprints:0402-res, symbol quicklogic-quick-feather-board:R_22R_0402
Connections:
- net labels added: ADC1, I2S_CLK, I2S_DOUT, I2S_WCLK, PDM_CKO, PDM_DATA, S3IO_10, S3IO_11, S3IO_12, S3IO_13, S3IO_2, S3IO_25, S3IO_27, S3IO_32_I2C1, S3IO_33_I2C1, S3IO_35_SPI_MST_CS3, S3IO_4, S3IO_40, S3IO_5, S3IO_7, S3IO_8, S3IO_9, S3_USB_D_N, S3_USB_D_P, SPI_MST_CS2, SPI_SLV_CLK, SPI_SLV_CSn, SPI_SLV_MISO, SPI_SLV_MOSI
- net labels removed: HEADER_MISO, HEADER_MOSI, MIC_CLOCK, MIC_DATA
- wire segments 317 -> 399
- no-connect marks 22 -> 4
Other:
- moved on the sheet: C1, C12, C13, C15, C17, C3, C4, C9, D1, D11, D5, J2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

Commit message: Component placement refined after pinout changes
Parts:
- removed R27: R_22R_0402, quicklogic-quick-feather-board-footprints:0402-res, symbol quicklogic-quick-feather-board:R_22R_0402
- removed TP4, TP5: TP_SMD1MM, quicklogic-quick-feather-board-footprints:Testpoint_smd_1mm, symbol quicklogic-quick-feather-board:TP_SMD1MM
- added TP4, TP5: TP_THT, quicklogic-quick-feather-board-footprints:Testpoint_THT_Drill0.9mm, symbol quicklogic-quick-feather-board:TP_THT
Connections:
- net labels added: J8.1, J8.10, J8.11, J8.12, J8.13, J8.14, J8.2, J8.3, J8.4, J8.5, J8.6, J8.7, J8.8, J8.9
- net labels removed: HEADER_SCK
- wire segments 399 -> 411
Other:
- note added: "const"
- moved on the sheet: J2, R33, R38, R39, R40, R41, R42
