File: quick-feather-board.sch (KiCad schematic (older format))
At the start: 99 parts, among them IC1 EOS-S3-QFN, J1 61300211121, J2 1x12_pinhead, J3 1x16_pinhead, J4 S2B-PH-SM4-TB_LF__SN_, J5 0473460001, J6 FTSH-105-01-L-DV-K, J7 61300211121, J8 2x8_pinhead, M1 mounting_pad, M2 mounting_pad, M3 mounting_pad, M4 mounting_pad, Q1 NX3008CBKV, Q2 2N7002PV, Q3 2N7002PV, U1 TPS62821DLCR, U2 MCP73831T-2ACI_OT, U3 GD25Q16CWIGR, U4 DPS310, U5 MC3635, X1 ECS-_327-12_5-34B-TR

Commit message: Re-generated production files
Parts:
- IC1: footprint quicklogic-quick-feather-board-footprints:QFN-64_EP_8.5x8.5_EOS -> quicklogic-quick-feather-board-footprints:QFN-64_8.5x8.5_EOS; MPN (none) -> EOSA1-S-PUN64; Manufacturer (none) -> QuickLogic
Changed lines of the file:
@@
 EESchema Schematic File Version 4
-LIBS:quicklogic-quick-feather-board-cache
 EELAYER 30 0
 EELAYER END
@@
 F 0 "IC1" H 3350 2230 50  0000 C CNN
 F 1 "EOS-S3-QFN" H 3540 2150 50  0000 C CNN
-F 2 "quicklogic-quick-feather-board-footprints:QFN-64_EP_8.5x8.5_EOS" H 4250 -1900 50  0001 C CNN
+F 2 "quicklogic-quick-feather-board-footprints:QFN-64_8.5x8.5_EOS" H 4250 -1900 50  0001 C CNN
 F 3 "" H 5050 -1600 50  0001 C CNN
+F 4 "EOSA1-S-PUN64" H 3300 1400 50  0001 C CNN "MPN"
+F 5 "QuickLogic" H 3300 1400 50  0001 C CNN "Manufacturer"
 	1    3300 1400
 	1    0    0    -1
