File: quick-feather-board.sch (KiCad schematic (older format))
At the start: 99 parts, among them IC1 EOS-S3-QFN, J1 61300211121, J2 1x12_pinhead, J3 1x16_pinhead, J4 S2B-PH-SM4-TB_LF__SN_, J5 0473460001, J6 FTSH-105-01-L-DV-K, J7 61300211121, J8 2x8_pinhead, M1 mounting_pad, M2 mounting_pad, M3 mounting_pad, M4 mounting_pad, Q1 NX3008CBKV, Q2 2N7002PV, Q3 2N7002PV, U1 TPS62821DLCR, U2 MCP73831T-2ACI_OT, U3 GD25Q16CWIGR, U4 DPS310, U5 MC3635, X1 ECS-_327-12_5-34B-TR

Commit message: Added delayed start circuit to battery charger
Parts:
- removed R1: R_100k_0402, quicklogic-quick-feather-board-footprints:0402-res, symbol quicklogic-quick-feather-board:R_100k_0402
- added C19: C_1u_0402, antmicro-footprints:0402-cap, symbol antmicroCapacitors0402:C_1u_0402
- added Q4: DMG1012T-7, antmicro-footprints:SOT-523, symbol antmicroTransistorsFETsMOSFETsSingle:DMG1012T-7
- added R1: R_1M8_0402, antmicro-footprints:0402-res, symbol antmicroResistors0402:R_1M8_0402
Connections:
- net labels added: PG
- wire segments 411 -> 413
Changed lines of the file:
@@
 $EndComp
 $Comp
-L quicklogic-quick-feather-board:R_100k_0402 R1
-U 1 1 5DC19E95
-P 1750 9100
-F 0 "R1" H 1750 9313 60  0000 C CNN
-F 1 "R_100k_0402" H 1750 8950 60  0001 C CNN
-F 2 "quicklogic-quick-feather-board-footprints:0402-res" H 1950 9300 60  0001 L CNN
-F 3 "" H 1750 9100 50  0001 C CNN
-F 4 "VISHAY" H 1950 9500 60  0001 L CNN "Manufacturer"
-F 5 "CRCW0402100KFKEDHP" H 1950 9400 60  0001 L CNN "MPN"
-F 6 "100k" H 1750 9215 50  0000 C CNN "Val"
-	1    1750 9100
-	1    0    0    -1
-$EndComp
-$Comp
 L quicklogic-quick-feather-board:GND #PWR0102
 U 1 1 5DC19F48
@@
 Connection ~ 1250 8800
 Wire Wire Line
-	1250 8800 950  8800
-Wire Wire Line
-	2250 9100 1900 9100
-Wire Wire Line
-	1600 9100 1550 9100
-Wire Wire Line
-	1550 9100 1550 8800
+	1250 8800 925  8800
 Wire Wire Line
 	2250 8950 2000 8950
@@
 L quicklogic-quick-feather-board:GND #PWR0106
 U 1 1 5DC1EFA0
-P 1950 6950
-F 0 "#PWR0106" H 1950 6700 50  0001 C CNN
-F 1 "GND" H 1955 6777 50  0000 C CNN
-F 2 "" H 1950 6950 50  0001 C CNN
-F 3 "" H 1950 6950 50  0001 C CNN
-	1    1950 6950
+P 1950 7350
+F 0 "#PWR0106" H 1950 7100 50  0001 C CNN
+F 1 "GND" H 1955 7177 50  0000 C CNN
+F 2 "" H 1950 7350 50  0001 C CNN
+F 3 "" H 1950 7350 50  0001 C CNN
+	1    1950 7350
 	1    0    0    -1
 $EndComp
@@
 L quicklogic-quick-feather-board:GND #PWR0107
 U 1 1 5DC1EFC3
-P 2750 6950
-F 0 "#PWR0107" H 2750 6700 50  0001 C CNN
-F 1 "GND" H 2755 6777 50  0000 C CNN
-F 2 "" H 2750 6950 50  0001 C CNN
-F 3 "" H 2750 6950 50  0001 C CNN
-	1    2750 6950
+P 2750 7325
+F 0 "#PWR0107" H 2750 7075 50  0001 C CNN
+F 1 "GND" H 2755 7152 50  0000 C CNN
+F 2 "" H 2750 7325 50  0001 C CNN
+F 3 "" H 2750 7325 50  0001 C CNN
+	1    2750 7325
 	1    0    0    -1
 $EndComp
 Wire Wire Line
 	1950 6850 1950 6950
-Wire Wire Line
-	2750 6850 2750 6950
 Text Notes 950  6750 0    50   ~ 0
 212mA charge current
@@
 Connection ~ 4900 8800
 Wire Wire Line
-	950  8800 950  8400
+	925  8800 925  8400
 Wire Wire Line
 	4900 8400 4900 8800
@@
 L quicklogic-quick-feather-board:+VBUS #PWR0123
 U 1 1 5E029AF7
-P 950 8350
-F 0 "#PWR0123" H 950 8350 50  0001 C CNN
-F 1 "+VBUS" H 935 8473 50  0000 C CNN
-F 2 "" H 950 8350 50  0001 C CNN
-F 3 "" H 950 8350 50  0001 C CNN
-	1    950  8350
+P 925 8350
+F 0 "#PWR0123" H 925 8350 50  0001 C CNN
+F 1 "+VBUS" H 910 8473 50  0000 C CNN
+F 2 "" H 925 8350 50  0001 C CNN
+F 3 "" H 925 8350 50  0001 C CNN
+	1    925  8350
 	1    0    0    -1
 $EndComp
@@
 Wire Wire Line
 	2000 4150 2950 4150
-Wire Wire Line
-	2000 8800 1550 8800
 Connection ~ 2000 8800
-Wire Wire Line
-	1550 8800 1250 8800
-Connection ~ 1550 8800
 Wire Notes Line
 	5450 8000 8350 8000
@@
 Wire Wire Line
 	2000 4450 2950 4450
+$Comp
+L antmicroTransistorsFETsMOSFETsSingle:DMG1012T-7 Q4
+U 1 1 5E9BD0BB
+P 1950 7150
+F 0 "Q4" H 2058 7203 60  0000 L CNN
+F 1 "DMG1012T-7" H 2058 7097 60  0000 L CNN
+F 2 "antmicro-footprints:SOT-523" H 2150 7350 60  0001 L CNN
+F 3 "https://www.diodes.com/assets/Datasheets/ds31783.pdf" H 2150 7450 60  0001 L CNN
+F 4 "DMG1012T-7" H 2150 7650 60  0001 L CNN "MPN"
+F 5 "Diodes Incorporated" H 2150 8250 60  0001 L CNN "Manufacturer"
+	1    1950 7150
+	1    0    0    -1
+$EndComp
+Wire Wire Line
+	2750 6850 2750 7325
+$Comp
+L antmicroResistors0402:R_1M8_0402 R1
+U 1 1 5EA0A68F
+P 1675 8950
+F 0 "R1" V 1630 9020 60  0000 L CNN
+F 1 "R_1M8_0402" H 1675 8800 60  0001 C CNN
+F 2 "antmicro-footprints:0402-res" H 1875 9150 60  0001 L CNN
+F 3 "" H 1675 8950 50  0001 C CNN
+F 4 "Multicomp" H 1875 9350 60  0001 L CNN "Manufacturer"
+F 5 "MCMR04X185_JTL" H 1875 9250 60  0001 L CNN "MPN"
+F 6 "1M8" V 1728 9020 50  0000 L CNN "Val"
+	1    1675 8950
+	0    1    1    0
+$EndComp
+Wire Wire Line
+	1250 8800 1675 8800
+Connection ~ 1675 8800
+Wire Wire Line
+	1675 8800 2000 8800
+Wire Wire Line
+	925  9100 1675 9100
+Connection ~ 1675 9100
+Wire Wire Line
+	1675 9100 2250 9100
+Text Label 975  9100 0    50   ~ 0
+PG
+Text Label 975  7050 0    50   ~ 0
+PG
+$Comp
+L quicklogic-quick-feather-board:GND #PWR028
+U 1 1 5EA7B915
+P 1350 7350
+F 0 "#PWR028" H 1350 7100 50  0001 C CNN
+F 1 "GND" H 1355 7177 50  0000 C CNN
+F 2 "" H 1350 7350 50  0001 C CNN
+F 3 "" H 1350 7350 50  0001 C CNN
+	1    1350 7350
+	1    0    0    -1
+$EndComp
+Wire Wire Line
+	1650 7250 1650 7050
+Wire Wire Line
+	1650 7050 1350 7050
+$Comp
+L antmicroCapacitors0402:C_1u_0402 C19
+U 1 1 5EA747B1
+P 1350 7200
+F 0 "C19" H 1465 7245 60  0000 L CNN
+F 1 "C_1u_0402" H 1350 7050 60  0001 C CNN
+F 2 "antmicro-footprints:0402-cap" H 1550 7400 60  0001 L CNN
+F 3 "" H 1350 7200 50  0001 C CNN
+F 4 "TDK" H 1550 7600 60  0001 L CNN "Manufacturer"
+F 5 "C1005X6S1A105K050BC" H 1550 7500 60  0001 L CNN "MPN"
+F 6 "1u" H 1465 7147 50  0000 L CNN "Val"
+	1    1350 7200
+	1    0    0    -1
+$EndComp
+Wire Wire Line
+	1350 7050 925  7050
+Connection ~ 1350 7050
 $EndSCHEMATC

Commit message: Updated library references
Parts:
- C1, C14, C16, C2, C5: footprint quicklogic-quick-feather-board-footprints:0603-cap -> quick-feather-board-footprints:0603-cap; symbol quicklogic-quick-feather-board:C_4u7_0603 -> quick-feather-board:C_4u7_0603
- C10, C11, C12, C13, C15, C17, C18, C8, C9: footprint quicklogic-quick-feather-board-footprints:0402-cap -> quick-feather-board-footprints:0402-cap; symbol quicklogic-quick-feather-board:C_100n_0402_6V3 -> quick-feather-board:C_100n_0402_6V3
- C19: footprint antmicro-footprints:0402-cap -> quick-feather-board-footprints:0402-cap; symbol antmicroCapacitors0402:C_1u_0402 -> quick-feather-board:C_1u_0402
- C3: footprint quicklogic-quick-feather-board-footprints:0402-cap -> quick-feather-board-footprints:0402-cap; symbol quicklogic-quick-feather-board:C_100p_0402 -> quick-feather-board:C_100p_0402
- C4: footprint quicklogic-quick-feather-board-footprints:0603-cap -> quick-feather-board-footprints:0603-cap; symbol quicklogic-quick-feather-board:C_22u_0603 -> quick-feather-board:C_22u_0603
- C6, C7: footprint quicklogic-quick-feather-board-footprints:0402-cap -> quick-feather-board-footprints:0402-cap; symbol quicklogic-quick-feather-board:C_12p_0402 -> quick-feather-board:C_12p_0402
- D1: footprint quicklogic-quick-feather-board-footprints:SOD-123 -> quick-feather-board-footprints:SOD-123; symbol quicklogic-quick-feather-board:MBR0520LT1G -> quick-feather-board:MBR0520LT1G
- D11, D3, D5: footprint quicklogic-quick-feather-board-footprints:SOT-3 -> quick-feather-board-footprints:SOT-3; symbol quicklogic-quick-feather-board:TPD2EUSB30DRTR -> quick-feather-board:TPD2EUSB30DRTR
- D2: footprint quicklogic-quick-feather-board-footprints:LED_0603 -> quick-feather-board-footprints:LED_0603; symbol quicklogic-quick-feather-board:LG_L29K-G2J1-24-Z -> quick-feather-board:LG_L29K-G2J1-24-Z
- D4: footprint quicklogic-quick-feather-board-footprints:LED-PLCC4_3.2x2.8mm_B -> quick-feather-board-footprints:LED-PLCC4_3.2x2.8mm_B; symbol quicklogic-quick-feather-board:ASMB-MTB1-0A3A2 -> quick-feather-board:ASMB-MTB1-0A3A2
- D6: footprint quicklogic-quick-feather-board-footprints:SOD-323-SD05 -> quick-feather-board-footprints:SOD-323-SD05; symbol quicklogic-quick-feather-board:SD05C.TCT -> quick-feather-board:SD05C.TCT
- IC1: footprint quicklogic-quick-feather-board-footprints:QFN-64_8.5x8.5_EOS -> quick-feather-board-footprints:QFN-64_8.5x8.5_EOS; symbol quicklogic-quick-feather-board:EOS-S3-QFN -> quick-feather-board:EOS-S3-QFN
- J1, J7: footprint quicklogic-quick-feather-board-footprints:PinHeader_1x2_P2.54_Drill0.9mm -> quick-feather-board-footprints:PinHeader_1x2_P2.54_Drill0.9mm; symbol quicklogic-quick-feather-board:61300211121 -> quick-feather-board:61300211121
- J2: footprint quicklogic-quick-feather-board-footprints:1x12_pinhead -> quick-feather-board-footprints:1x12_pinhead; symbol quicklogic-quick-feather-board:1x12_pinhead -> quick-feather-board:1x12_pinhead
- J3: footprint quicklogic-quick-feather-board-footprints:1x16_pinhead -> quick-feather-board-footprints:1x16_pinhead; symbol quicklogic-quick-feather-board:1x16_pinhead -> quick-feather-board:1x16_pinhead
- J4: footprint quicklogic-quick-feather-board-footprints:PinHeader_2x1mm_P2mm_SMD_RA -> quick-feather-board-footprints:PinHeader_2x1mm_P2mm_SMD_RA; symbol quicklogic-quick-feather-board:S2B-PH-SM4-TB_LF__SN_ -> quick-feather-board:S2B-PH-SM4-TB_LF__SN_
- J5: footprint quicklogic-quick-feather-board-footprints:USB_Micro_B_Female_0473460001 -> quick-feather-board-footprints:USB_Micro_B_Female_0473460001; symbol quicklogic-quick-feather-board:0473460001 -> quick-feather-board:0473460001
- J6: footprint quicklogic-quick-feather-board-footprints:PinHeader_2x5_P1.27_SMD -> quick-feather-board-footprints:PinHeader_2x5_P1.27_SMD; symbol quicklogic-quick-feather-board:FTSH-105-01-L-DV-K -> quick-feather-board:FTSH-105-01-L-DV-K
- J8: footprint quicklogic-quick-feather-board-footprints:2x8_pinhead -> quick-feather-board-footprints:2x8_pinhead; symbol quicklogic-quick-feather-board:2x8_pinhead -> quick-feather-board:2x8_pinhead
- L1: footprint quicklogic-quick-feather-board-footprints:0806 -> quick-feather-board-footprints:0806; symbol quicklogic-quick-feather-board:DFE201610E-R47M=P2 -> quick-feather-board:DFE201610E-R47M=P2
- M1, M2, M3, M4: footprint quicklogic-quick-feather-board-footprints:MPAD -> quick-feather-board-footprints:MPAD; symbol quicklogic-quick-feather-board:mounting_pad -> quick-feather-board:mounting_pad
- MIC1: footprint quicklogic-quick-feather-board-footprints:IM69D130 -> quick-feather-board-footprints:IM69D130; symbol quicklogic-quick-feather-board:IM69D130 -> quick-feather-board:IM69D130
- N1: footprint quicklogic-quick-feather-board-footprints:oshw-logo -> quick-feather-board-footprints:oshw-logo; symbol quicklogic-quick-feather-board:oshw_logo -> quick-feather-board:oshw_logo
- N2: footprint quicklogic-quick-feather-board-footprints:LOGO -> quick-feather-board-footprints:LOGO; symbol quicklogic-quick-feather-board:ql_logo -> quick-feather-board:ql_logo
- Q1: footprint quicklogic-quick-feather-board-footprints:SOT-563 -> quick-feather-board-footprints:SOT-563; symbol quicklogic-quick-feather-board:NX3008CBKV -> quick-feather-board:NX3008CBKV
- Q2, Q3: footprint quicklogic-quick-feather-board-footprints:SOT-563 -> quick-feather-board-footprints:SOT-563; symbol quicklogic-quick-feather-board:2N7002PV -> quick-feather-board:2N7002PV
- Q4: footprint antmicro-footprints:SOT-523 -> quick-feather-board-footprints:SOT-523; symbol antmicroTransistorsFETsMOSFETsSingle:DMG1012T-7 -> quick-feather-board:DMG1012T-7
- R1: footprint antmicro-footprints:0402-res -> quick-feather-board-footprints:0402-res; symbol antmicroResistors0402:R_1M8_0402 -> quick-feather-board:R_1M8_0402
- R10, R14, R15, R19, R21, R22, R23, R31, R32, R34, R36, R37, R6, R8: footprint quicklogic-quick-feather-board-footprints:0402-res -> quick-feather-board-footprints:0402-res; symbol quicklogic-quick-feather-board:R_10k_0402 -> quick-feather-board:R_10k_0402
- R11, R28, R29, R35, R38, R39, R40, R7: footprint quicklogic-quick-feather-board-footprints:0402-res -> quick-feather-board-footprints:0402-res; symbol quicklogic-quick-feather-board:R_22R_0402 -> quick-feather-board:R_22R_0402
- R12, R17, R5: footprint quicklogic-quick-feather-board-footprints:0402-res -> quick-feather-board-footprints:0402-res; symbol quicklogic-quick-feather-board:R_100k_0402 -> quick-feather-board:R_100k_0402
- R13, R24, R26: footprint quicklogic-quick-feather-board-footprints:0402-res -> quick-feather-board-footprints:0402-res; symbol quicklogic-quick-feather-board:R_100R_0402 -> quick-feather-board:R_100R_0402
- R16: footprint quicklogic-quick-feather-board-footprints:0402-res -> quick-feather-board-footprints:0402-res; symbol quicklogic-quick-feather-board:R_200k_0402 -> quick-feather-board:R_200k_0402
- R18, R2, R20: footprint quicklogic-quick-feather-board-footprints:0402-res -> quick-feather-board-footprints:0402-res; symbol quicklogic-quick-feather-board:R_4k7_0402 -> quick-feather-board:R_4k7_0402
- R25: footprint quicklogic-quick-feather-board-footprints:0402-res -> quick-feather-board-footprints:0402-res; symbol quicklogic-quick-feather-board:R_220R_0402 -> quick-feather-board:R_220R_0402
- R3, R9: footprint quicklogic-quick-feather-board-footprints:0402-res -> quick-feather-board-footprints:0402-res; symbol quicklogic-quick-feather-board:R_1k5_0402 -> quick-feather-board:R_1k5_0402
- R30, R33, R41, R42: footprint quicklogic-quick-feather-board-footprints:R_Array_Convex_8x0602 -> quick-feather-board-footprints:R_Array_Convex_8x0602; symbol quicklogic-quick-feather-board:EXB2HV220JV -> quick-feather-board:EXB2HV220JV
- R4: footprint quicklogic-quick-feather-board-footprints:0402-res -> quick-feather-board-footprints:0402-res; symbol quicklogic-quick-feather-board:R_453k_0402 -> quick-feather-board:R_453k_0402
- S1, S2: footprint quicklogic-quick-feather-board-footprints:SW_SPST_4.2x2.8 -> quick-feather-board-footprints:SW_SPST_4.2x2.8; symbol quicklogic-quick-feather-board:KMR2 -> quick-feather-board:KMR2
- TP1, TP2, TP6: footprint quicklogic-quick-feather-board-footprints:Testpoint_smd_1mm -> quick-feather-board-footprints:Testpoint_smd_1mm; symbol quicklogic-quick-feather-board:TP_SMD1MM -> quick-feather-board:TP_SMD1MM
- TP4, TP5: footprint quicklogic-quick-feather-board-footprints:Testpoint_THT_Drill0.9mm -> quick-feather-board-footprints:Testpoint_THT_Drill0.9mm; symbol quicklogic-quick-feather-board:TP_THT -> quick-feather-board:TP_THT
- U1: footprint quicklogic-quick-feather-board-footprints:QFN-8_2x1mm -> quick-feather-board-footprints:QFN-8_2x1mm; symbol quicklogic-quick-feather-board:TPS62821DLCR -> quick-feather-board:TPS62821DLCR
- U2: footprint quicklogic-quick-feather-board-footprints:SOT-753 -> quick-feather-board-footprints:SOT-753; symbol quicklogic-quick-feather-board:MCP73831T-2ACI_OT -> quick-feather-board:MCP73831T-2ACI_OT
- U3: footprint quicklogic-quick-feather-board-footprints:GD25Q16CWIG -> quick-feather-board-footprints:GD25Q16CWIG; symbol quicklogic-quick-feather-board:GD25Q16CWIGR -> quick-feather-board:GD25Q16CWIGR
- U4: footprint quicklogic-quick-feather-board-footprints:PG-VLGA-8-2 -> quick-feather-board-footprints:PG-VLGA-8-2; symbol quicklogic-quick-feather-board:DPS310 -> quick-feather-board:DPS310
- U5: footprint quicklogic-quick-feather-board-footprints:MC3635 -> quick-feather-board-footprints:MC3635; symbol quicklogic-quick-feather-board:MC3635 -> quick-feather-board:MC3635
- X1: footprint quicklogic-quick-feather-board-footprints:SMD-2_3.2x1.5mm -> quick-feather-board-footprints:SMD-2_3.2x1.5mm; symbol quicklogic-quick-feather-board:ECS-_327-12_5-34B-TR -> quick-feather-board:ECS-_327-12_5-34B-TR

Commit message: Updated PCB layout for charger with delayed startup
Parts:
- removed R1: R_1M8_0402, quick-feather-board-footprints:0402-res, symbol quick-feather-board:R_1M8_0402
- removed R35: R_22R_0402, quick-feather-board-footprints:0402-res, symbol quick-feather-board:R_22R_0402
- added R1: R_1M5_0402, antmicro-footprints:0402-res, symbol antmicroResistors0402:R_1M5_0402
Connections:
- net labels removed: HEADER_A5
- wire segments 413 -> 411
Changed lines of the file:
@@
 F 3 "" H 1250 9300 50  0001 C CNN
 	1    1250 9300
-	1    0    0    -1
+	0    1    1    0
 $EndComp
 Wire Wire Line
@@
 USB_D_P
 $Comp
-L quick-feather-board:R_22R_0402 R7
-U 1 1 5DE231E1
-P 2160 4350
-F 0 "R7" H 2160 4563 60  0000 C CNN
-F 1 "R_22R_0402" H 2160 4200 60  0001 C CNN
-F 2 "quick-feather-board-footprints:0402-res" H 2360 4550 60  0001 L CNN
-F 3 "" H 2160 4350 50  0001 C CNN
-F 4 "VISHAY" H 2360 4750 60  0001 L CNN "Manufacturer"
-F 5 "CRCW040222R0FKED" H 2360 4650 60  0001 L CNN "MPN"
-F 6 "22R" H 2160 4465 50  0000 C CNN "Val"
-	1    2160 4350
-	-1   0    0    -1
-$EndComp
-$Comp
 L quick-feather-board:R_22R_0402 R11
 U 1 1 5DE232D3
@@
 $EndComp
 Wire Wire Line
-	2000 4350 1250 4350
-Wire Wire Line
 	1700 4450 1600 4450
 $Comp
@@
 Wire Wire Line
 	9800 6750 9800 6650
-Connection ~ 9800 6650
-Wire Wire Line
-	9800 6650 9800 6300
-Wire Wire Line
-	9800 6000 9300 6000
-Text Label 9300 6000 0    50   ~ 0
-HEADER_A5
 Wire Wire Line
 	9800 7050 9800 7100
@@
 Connection ~ 10050 7000
 Connection ~ 4400 6450
-$Comp
-L quick-feather-board:R_22R_0402 R35
-U 1 1 5E34140B
-P 9800 6150
-F 0 "R35" V 9850 6000 60  0000 C CNN
-F 1 "R_22R_0402" H 9800 6000 60  0001 C CNN
-F 2 "quick-feather-board-footprints:0402-res" H 10000 6350 60  0001 L CNN
-F 3 "" H 9800 6150 50  0001 C CNN
-F 4 "VISHAY" H 10000 6550 60  0001 L CNN "Manufacturer"
-F 5 "CRCW040222R0FKED" H 10000 6450 60  0001 L CNN "MPN"
-F 6 "22R" V 9750 6000 50  0000 C CNN "Val"
-F 7 "1" V 9800 6150 50  0001 C CNN "DNP"
-	1    9800 6150
-	0    1    -1   0
-$EndComp
-Text Notes 9400 6200 0    50   ~ 10
-DNP
 Text Notes 9400 6950 0    50   ~ 10
 DNP
@@
 Wire Wire Line
 	2750 6850 2750 7325
-$Comp
-L quick-feather-board:R_1M8_0402 R1
-U 1 1 5EA0A68F
-P 1675 8950
-F 0 "R1" V 1630 9020 60  0000 L CNN
-F 1 "R_1M8_0402" H 1675 8800 60  0001 C CNN
-F 2 "quick-feather-board-footprints:0402-res" H 1875 9150 60  0001 L CNN
-F 3 "" H 1675 8950 50  0001 C CNN
-F 4 "Multicomp" H 1875 9350 60  0001 L CNN "Manufacturer"
-F 5 "MCMR04X185_JTL" H 1875 9250 60  0001 L CNN "MPN"
-F 6 "1M8" V 1728 9020 50  0000 L CNN "Val"
-	1    1675 8950
-	0    1    1    0
-$EndComp
-Wire Wire Line
-	1250 8800 1675 8800
-Connection ~ 1675 8800
-Wire Wire Line
-	1675 8800 2000 8800
-Wire Wire Line
-	925  9100 1675 9100
-Connection ~ 1675 9100
-Wire Wire Line
-	1675 9100 2250 9100
 Text Label 975  9100 0    50   ~ 0
 PG
@@
 	1350 7050 925  7050
 Connection ~ 1350 7050
+$Comp
+L quick-feather-board:R_22R_0402 R7
+U 1 1 5DE231E1
+P 2160 4350
+F 0 "R7" H 2160 4563 60  0000 C CNN
+F 1 "R_22R_0402" H 2160 4200 60  0001 C CNN
+F 2 "quick-feather-board-footprints:0402-res" H 2360 4550 60  0001 L CNN
+F 3 "" H 2160 4350 50  0001 C CNN
+F 4 "VISHAY" H 2360 4750 60  0001 L CNN "Manufacturer"
+F 5 "CRCW040222R0FKED" H 2360 4650 60  0001 L CNN "MPN"
+F 6 "22R" H 2160 4465 50  0000 C CNN "Val"
+	1    2160 4350
+	-1   0    0    -1
+$EndComp
+Wire Wire Line
+	2010 4350 1244 4350
+$Comp
+L antmicroResistors0402:R_1M5_0402 R1
+U 1 1 5E8E2484
+P 1650 8950
+F 0 "R1" V 1605 9020 60  0000 L CNN
+F 1 "R_1M5_0402" H 1650 8800 60  0001 C CNN
+F 2 "antmicro-footprints:0402-res" H 1850 9150 60  0001 L CNN
+F 3 "" H 1650 8950 50  0001 C CNN
+F 4 "Multicomp" H 1850 9350 60  0001 L CNN "Manufacturer"
+F 5 "MCWR04W1504FTL" H 1850 9250 60  0001 L CNN "MPN"
+F 6 "1M5" V 1703 9020 50  0000 L CNN "Val"
+	1    1650 8950
+	0    1    1    0
+$EndComp
+Wire Wire Line
+	1250 8800 1650 8800
+Wire Wire Line
+	925  9100 1650 9100
+Connection ~ 1650 8800
+Wire Wire Line
+	1650 8800 2000 8800
+Connection ~ 1650 9100
+Wire Wire Line
+	1650 9100 2250 9100
 $EndSCHEMATC

Commit message: BOM and internal library updated
Parts:
- R1: footprint antmicro-footprints:0402-res -> quick-feather-board-footprints:0402-res; symbol antmicroResistors0402:R_1M5_0402 -> quick-feather-board:R_1M5_0402
Changed lines of the file:
@@
 	2010 4350 1244 4350
 $Comp
-L antmicroResistors0402:R_1M5_0402 R1
+L quick-feather-board:R_1M5_0402 R1
 U 1 1 5E8E2484
 P 1650 8950
 F 0 "R1" V 1605 9020 60  0000 L CNN
 F 1 "R_1M5_0402" H 1650 8800 60  0001 C CNN
-F 2 "antmicro-footprints:0402-res" H 1850 9150 60  0001 L CNN
+F 2 "quick-feather-board-footprints:0402-res" H 1850 9150 60  0001 L CNN
 F 3 "" H 1650 8950 50  0001 C CNN
 F 4 "Multicomp" H 1850 9350 60  0001 L CNN "Manufacturer"

Commit message: Corrected IO_27 to IO_30
Connections:
- net labels added: S3IO_30
- net labels removed: S3IO_27
Changed lines of the file:
@@
 PDM_CKO
 Text Label 5500 3450 0    50   ~ 0
-S3IO_27
+S3IO_30
 Text Label 13000 3100 0    50   ~ 0
-S3IO_27
+S3IO_30
 Text Label 5500 3550 0    50   ~ 0
 I2S_CLK
