File: quickfeather-board.sch (KiCad schematic (older format))
At the start: 100 parts, among them IC1 EOS-S3-QFN, J1 61300211121, J2 1x12_pinhead, J3 1x16_pinhead, J4 S2B-PH-SM4-TB_LF__SN_, J5 0473460001, J6 FTSH-105-01-L-DV-K, J7 61300211121, J8 2x8_pinhead, M1 mounting_pad, M2 mounting_pad, M3 mounting_pad, M4 mounting_pad, Q1 NX3008CBKV, Q2 2N7002PV, Q3 2N7002PV, Q4 DMG1012T-7, U1 TPS62821DLCR, U2 MCP73831T-2ACI_OT, U3 GD25Q16CWIGR, U4 DPS310, U5 MC3635, X1 ECS-_327-12_5-34B-TR

Commit message: Add release 1.2.0
Parts:
- added R27: R_1k5_0402, quickfeather-board-footprints:0402-res, symbol quickfeather-board:R_1k5_0402
Connections:
- wire segments 411 -> 417
Changed lines of the file:
@@
 Title "QuickFeather Development Kit"
 Date ""
-Rev "1.1"
+Rev "1.2.0"
 Comp ""
 Comment1 "www.antmicro.com"
@@
 U 1 1 5DE232D3
 P 1850 4450
-F 0 "R11" H 1850 4250 60  0000 C CNN
+F 0 "R11" H 1600 4500 60  0000 C CNN
 F 1 "R_22R_0402" H 1850 4300 60  0001 C CNN
 F 2 "quickfeather-board-footprints:0402-res" H 2050 4650 60  0001 L CNN
@@
 F 4 "VISHAY" H 2050 4850 60  0001 L CNN "Manufacturer"
 F 5 "CRCW040222R0FKED" H 2050 4750 60  0001 L CNN "MPN"
-F 6 "22R" H 1850 4350 50  0000 C CNN "Val"
+F 6 "22R" H 1850 4450 50  0000 C CNN "Val"
 	1    1850 4450
 	-1   0    0    -1
@@
 L quickfeather-board:R_1k5_0402 R9
 U 1 1 5DE457DE
-P 1850 4150
-F 0 "R9" H 2050 4200 60  0000 C CNN
-F 1 "R_1k5_0402" H 1850 4000 60  0001 C CNN
-F 2 "quickfeather-board-footprints:0402-res" H 2050 4350 60  0001 L CNN
-F 3 "" H 1850 4150 50  0001 C CNN
-F 4 "PANASONIC_ELECTRONIC_COMPONENTS" H 2050 4550 60  0001 L CNN "Manufacturer"
-F 5 "ERJ2RKF1501X" H 2050 4450 60  0001 L CNN "MPN"
-F 6 "1k5" H 1850 4050 50  0000 C CNN "Val"
-	1    1850 4150
+P 1850 4675
+F 0 "R9" H 1625 4725 60  0000 C CNN
+F 1 "R_1k5_0402" H 1850 4525 60  0001 C CNN
+F 2 "quickfeather-board-footprints:0402-res" H 2050 4875 60  0001 L CNN
+F 3 "" H 1850 4675 50  0001 C CNN
+F 4 "PANASONIC_ELECTRONIC_COMPONENTS" H 2050 5075 60  0001 L CNN "Manufacturer"
+F 5 "ERJ2RKF1501X" H 2050 4975 60  0001 L CNN "MPN"
+F 6 "1k5" H 1850 4675 50  0000 C CNN "Val"
+	1    1850 4675
 	-1   0    0    -1
 $EndComp
@@
 	1600 4450 1250 4450
 Wire Wire Line
-	1600 4150 1600 4450
-Wire Wire Line
 	1600 4150 1700 4150
 Wire Wire Line
@@
 	2950 4250 2420 4250
 Wire Wire Line
-	2950 4350 2310 4350
+	2950 4350 2010 4350
 Text Label 5500 3050 0    50   ~ 0
 I2S_DOUT
@@
 	5000 3350 6300 3350
 Wire Wire Line
-	2000 4150 2950 4150
+	2000 4150 2250 4150
 Connection ~ 2000 8800
 Wire Notes Line
@@
 	690  700  8350 700
 Wire Wire Line
-	2950 4050 2100 4050
+	2950 4050 1750 4050
 $Comp
 L quickfeather-board:TP_THT TP5
 U 1 1 5F03C1C3
-P 2000 4050
-F 0 "TP5" V 2000 3950 50  0000 C CNN
-F 1 "TP_THT" H 2000 3950 50  0001 C CNN
-F 2 "quickfeather-board-footprints:Testpoint_THT_Drill0.9mm" H 2200 4250 60  0001 L CNN
-F 3 "" H 2200 4350 60  0001 L CNN
-F 4 "N/A" H 2000 4050 50  0001 C CNN "Manufacturer"
-F 5 "N/A" H 2000 4050 50  0001 C CNN "MPN"
-	1    2000 4050
+P 1650 4050
+F 0 "TP5" V 1650 3950 50  0000 C CNN
+F 1 "TP_THT" H 1650 3950 50  0001 C CNN
+F 2 "quickfeather-board-footprints:Testpoint_THT_Drill0.9mm" H 1850 4250 60  0001 L CNN
+F 3 "" H 1850 4350 60  0001 L CNN
+F 4 "N/A" H 1650 4050 50  0001 C CNN "Manufacturer"
+F 5 "N/A" H 1650 4050 50  0001 C CNN "MPN"
+	1    1650 4050
 	0    1    1    0
 $EndComp
@@
 L quickfeather-board:R_22R_0402 R7
 U 1 1 5DE231E1
-P 2160 4350
-F 0 "R7" H 2160 4563 60  0000 C CNN
-F 1 "R_22R_0402" H 2160 4200 60  0001 C CNN
-F 2 "quickfeather-board-footprints:0402-res" H 2360 4550 60  0001 L CNN
-F 3 "" H 2160 4350 50  0001 C CNN
-F 4 "VISHAY" H 2360 4750 60  0001 L CNN "Manufacturer"
-F 5 "CRCW040222R0FKED" H 2360 4650 60  0001 L CNN "MPN"
-F 6 "22R" H 2160 4465 50  0000 C CNN "Val"
-	1    2160 4350
+P 1860 4350
+F 0 "R7" H 1645 4400 60  0000 C CNN
+F 1 "R_22R_0402" H 1860 4200 60  0001 C CNN
+F 2 "quickfeather-board-footprints:0402-res" H 2060 4550 60  0001 L CNN
+F 3 "" H 1860 4350 50  0001 C CNN
+F 4 "VISHAY" H 2060 4750 60  0001 L CNN "Manufacturer"
+F 5 "CRCW040222R0FKED" H 2060 4650 60  0001 L CNN "MPN"
+F 6 "22R" H 1870 4350 50  0000 C CNN "Val"
+	1    1860 4350
 	-1   0    0    -1
 $EndComp
 Wire Wire Line
-	2010 4350 1244 4350
+	1710 4350 1600 4350
 $Comp
 L quickfeather-board:R_1M5_0402 R1
@@
 Wire Wire Line
 	1650 9100 2250 9100
+Text Notes 15250 5950 2    51   ~ 10
+DNP
+$Comp
+L quickfeather-board:R_1k5_0402 R27
+U 1 1 5EBB0A85
+P 1850 4150
+F 0 "R27" H 1600 4200 60  0000 C CNN
+F 1 "R_1k5_0402" H 1850 4000 60  0001 C CNN
+F 2 "quickfeather-board-footprints:0402-res" H 2050 4350 60  0001 L CNN
+F 3 "" H 1850 4150 50  0001 C CNN
+F 4 "PANASONIC_ELECTRONIC_COMPONENTS" H 2050 4550 60  0001 L CNN "Manufacturer"
+F 5 "ERJ2RKF1501X" H 2050 4450 60  0001 L CNN "MPN"
+F 6 "1k5" H 1850 4150 50  0000 C CNN "Val"
+F 7 "1" H 1850 4150 50  0001 C CNN "DNP"
+	1    1850 4150
+	-1   0    0    -1
+$EndComp
+Wire Wire Line
+	1600 4450 1600 4675
+Wire Wire Line
+	1600 4675 1700 4675
+Wire Wire Line
+	2000 4675 2250 4675
+Wire Wire Line
+	2250 4675 2250 4150
+Connection ~ 2250 4150
+Wire Wire Line
+	2250 4150 2950 4150
+Wire Wire Line
+	1600 4150 1600 4350
+Connection ~ 1600 4350
+Wire Wire Line
+	1600 4350 1244 4350
+Text Notes 2175 4225 2    51   ~ 10
+DNP
 $EndSCHEMATC

Commit message: Add release 1.2.1
Parts:
- R27: DNP 1 -> (none)
Connections:
- net labels added: PU_CTRL_USBN
- net labels removed: S3IO_40
- wire segments 417 -> 416
Changed lines of the file:
@@
 Title "QuickFeather Development Kit"
 Date ""
-Rev "1.2.0"
+Rev "1.2.1"
 Comp ""
 Comment1 "www.antmicro.com"
@@
 	2950 3950 2390 3950
 Wire Wire Line
-	2950 4250 2420 4250
-Wire Wire Line
 	2950 4350 2010 4350
 Text Label 5500 3050 0    50   ~ 0
@@
 Text Label 13000 3700 0    50   ~ 0
 SPI_MST_MISO
-Text Label 2370 4150 0    50   ~ 0
-PU_CTRL_USBP
 Text Label 13000 3600 0    50   ~ 0
 SPI_MST_MOSI
-Text Label 2450 4250 0    50   ~ 0
-S3IO_40
-Text Label 2450 4350 0    50   ~ 0
-S3_USB_D_N
 Text Label 2350 4450 0    50   ~ 0
 S3_USB_D_P
@@
 Wire Wire Line
 	5000 3350 6300 3350
-Wire Wire Line
-	2000 4150 2250 4150
 Connection ~ 2000 8800
 Wire Notes Line
@@
 Text Label 13400 6650 2    50   ~ 0
 PDM_CKO
-Text Label 14950 7050 2    50   ~ 0
-S3IO_40
 Wire Wire Line
 	13050 6650 13450 6650
@@
 Wire Wire Line
 	14600 6850 15000 6850
-Wire Wire Line
-	14600 7050 15000 7050
 Text Label 14650 6550 0    50   ~ 0
 S3IO_5
@@
 Wire Wire Line
 	15350 6850 15550 6850
-Wire Wire Line
-	15350 7050 15550 7050
 Text Label 13850 6650 0    50   ~ 0
 J8.2
@@
 Text Label 15400 6850 0    50   ~ 0
 J8.12
-Text Label 15400 7050 0    50   ~ 0
-J8.14
 Text Notes 12850 5750 0    50   ~ 0
 const
@@
 F 5 "ERJ2RKF1501X" H 2050 4450 60  0001 L CNN "MPN"
 F 6 "1k5" H 1850 4150 50  0000 C CNN "Val"
-F 7 "1" H 1850 4150 50  0001 C CNN "DNP"
 	1    1850 4150
 	-1   0    0    -1
@@
 	2000 4675 2250 4675
 Wire Wire Line
-	2250 4675 2250 4150
-Connection ~ 2250 4150
-Wire Wire Line
-	2250 4150 2950 4150
-Wire Wire Line
 	1600 4150 1600 4350
 Connection ~ 1600 4350
 Wire Wire Line
 	1600 4350 1244 4350
-Text Notes 2175 4225 2    51   ~ 10
-DNP
+Text Label 2450 4350 0    50   ~ 0
+S3_USB_D_N
+Text Label 2350 4250 0    50   ~ 0
+PU_CTRL_USBN
+Text Label 2350 4150 0    50   ~ 0
+PU_CTRL_USBP
+Wire Wire Line
+	2950 4150 2250 4150
+Wire Wire Line
+	2250 4150 2250 4675
+Wire Wire Line
+	2950 4250 2150 4250
+Wire Wire Line
+	2150 4250 2150 4150
+Wire Wire Line
+	2150 4150 2000 4150
 $EndSCHEMATC
